File: PCB/Gantry_PCBv2/Gantry_PCBv2.kicad_sch (KiCad schematic)
At the start: 169 parts, among them J1 Screw_Terminal_01x02, J10 B2B-XH-A_LF__SN_, J11 USB_C_Receptacle_USB2.0_16P, J12 Conn_01x04_Pin, J13 Conn_01x04_Pin, J14 Conn_01x04_Pin, J15 Conn_01x04_Pin, J16 Conn_01x05_Pin, J17 Conn_01x05_Pin, J2 DCJ200-10-A-XX-X_REVA, J3 Conn_01x03_Pin, J4 Conn_01x14, J5 B2B-XH-A_LF__SN_, J6 B2B-XH-A_LF__SN_, J7 B2B-XH-A_LF__SN_, J8 Conn_01x14, J9 Conn_01x10, Q1 NMOS, Q2 SS8050, Q3 SS8050, SW1 SW_0, SW2 SW_EN, SW3 SW_Push_DPDT, SW4 SW_Push_DPDT, SW5 SW_Push_DPDT, SW6 SW_Push_DPDT, U10 74HC245, U11 74HC245, U12 MCP23017_SO, U13 CP2102N-Axx-xQFN28, U14 ESP32-WROOM-32U, U2 MP1584, U4 TLV75733PDBV, U5 DRV8825_STEPPER_MOTOR_DRIVER_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, U6 DRV8825_STEPPER_MOTOR_DRIVER_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, U7 TB6612FNG H-bridge Motor Driv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, U8 DRV8825_STEPPER_MOTOR_DRIVER_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, U9 DRV8825_STEPPER_MOTOR_DRIVER_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

Commit message: PCB routing 1st draft
Connections:
- net SM1_A1: now also J15.2 (Pin_2); no longer J15.1 (Pin_1)
- net SM1_A2: now also J15.1 (Pin_1); no longer J15.2 (Pin_2)
- net SM2_A1: now also J12.2 (Pin_2); no longer J12.1 (Pin_1)
- net SM2_A2: now also J12.1 (Pin_1); no longer J12.2 (Pin_2)
- net SM3_A1: now also J13.2 (Pin_2); no longer J13.1 (Pin_1)
- net SM3_A2: now also J13.1 (Pin_1); no longer J13.2 (Pin_2)
- net SM4_A1: now also J14.2 (Pin_2); no longer J14.1 (Pin_1)
- net SM4_A2: now also J14.1 (Pin_1); no longer J14.2 (Pin_2)
Changed lines of the file:
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@@
 		)
 	)
-	(label "SM4_A1"
+	(label "SM4_A2"
 		(at 246.888 270.256 0)
 		(effects
@@
 		)
 	)
-	(label "SM2_A2"
+	(label "SM2_A1"
 		(at 208.788 272.796 0)
 		(effects
@@
 		)
 	)
-	(label "SM2_A1"
+	(label "SM2_A2"
 		(at 208.788 270.256 0)
 		(effects
@@
 		)
 	)
-	(label "SM4_A2"
+	(label "SM4_A1"
 		(at 246.888 272.796 0)
 		(effects
@@
 		)
 	)
-	(label "SM1_A1"
+	(label "SM1_A2"
 		(at 267.208 270.256 0)
 		(effects
@@
 		)
 	)
-	(label "SM1_A2"
+	(label "SM1_A1"
 		(at 267.208 272.796 0)
 		(effects
@@
 		)
 	)
-	(label "SM3_A1"
+	(label "SM3_A2"
 		(at 229.108 270.256 0)
 		(effects
@@
 		)
 	)
-	(label "SM3_A2"
+	(label "SM3_A1"
 		(at 229.108 272.796 0)
 		(effects
